File: rev1/FTRM60.kicad_pcb (KiCad board)
At the start: 2 copper layers, 285.2 x 99.8 mm, 152 parts, among them J1 SM04B-SRSS-TB(LF)(SN), U2 ATmega32U4-AU, Y1 16MHz

Commit message: Some late updates
Parts:
- removed REF** (x4): MountingHole_2.2mm_M2_Pad, MountingHole:MountingHole_2.2mm_M2_Pad
Routing:
- net Net-(D58-Pad2): track 18.5 -> 16.9 mm
Changed lines of the file:
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@@
     (thickness 1.6)
     (drawings 30)
-    (tracks 707)
+    (tracks 710)
     (zones 0)
-    (modules 152)
+    (modules 148)
     (nets 101)
   )
@@
     (solder_mask_min_width 0.25)
     (aux_axis_origin 0 0)
-    (visible_elements 7FFFEFFF)
+    (visible_elements 7FFFFFFF)
     (pcbplotparams
       (layerselection 0x010fc_ffffffff)
@@
     (add_net GND)
   )
-  (module MountingHole:MountingHole_2.2mm_M2_Pad (layer F.Cu)
-    (at 338.93125 101.6)
-    (descr "Mounting Hole 2.2mm, M2")
-    (tags "mounting hole 2.2mm m2")
-    (attr virtual)
-    (fp_text reference REF** (at 0 -3.2) (layer F.SilkS) hide
-      (effects (font (size 1 1) (thickness 0.15)))
-    )
-    (fp_text value MountingHole_2.2mm_M2_Pad (at 0 3.2) (layer F.Fab)
-      (effects (font (size 1 1) (thickness 0.15)))
-    )
-    (fp_circle (center 0 0) (end 2.45 0) (layer F.CrtYd) (width 0.05))
-    (fp_circle (center 0 0) (end 2.2 0) (layer Cmts.User) (width 0.15))
-    (fp_text user %R (at 0.3 0) (layer F.Fab)
-      (effects (font (size 1 1) (thickness 0.15)))
-    )
-    (pad 1 thru_hole circle (at 0 0) (size 4.4 4.4) (drill 2.2) (layers *.Cu *.Mask))
-  )
-  (module MountingHole:MountingHole_2.2mm_M2_Pad (layer F.Cu)
-    (at 340.51875 156.36875)
-    (descr "Mounting Hole 2.2mm, M2")
-    (tags "mounting hole 2.2mm m2")
-    (attr virtual)
-    (fp_text reference REF** (at 0 -3.2) (layer F.SilkS) hide
-      (effects (font (size 1 1) (thickness 0.15)))
-    )
-    (fp_text value MountingHole_2.2mm_M2_Pad (at 0 3.2) (layer F.Fab)
-      (effects (font (size 1 1) (thickness 0.15)))
-    )
-    (fp_circle (center 0 0) (end 2.45 0) (layer F.CrtYd) (width 0.05))
-    (fp_circle (center 0 0) (end 2.2 0) (layer Cmts.User) (width 0.15))
-    (fp_text user %R (at 0.3 0) (layer F.Fab)
-      (effects (font (size 1 1) (thickness 0.15)))
-    )
-    (pad 1 thru_hole circle (at 0 0) (size 4.4 4.4) (drill 2.2) (layers *.Cu *.Mask))
-  )
-  (module MountingHole:MountingHole_2.2mm_M2_Pad (layer F.Cu)
-    (at 103.1875 155.575)
-    (descr "Mounting Hole 2.2mm, M2")
-    (tags "mounting hole 2.2mm m2")
-    (attr virtual)
-    (fp_text reference REF** (at 0 -3.2) (layer F.SilkS) hide
-      (effects (font (size 1 1) (thickness 0.15)))
-    )
-    (fp_text value MountingHole_2.2mm_M2_Pad (at 0 3.2) (layer F.Fab)
-      (effects (font (size 1 1) (thickness 0.15)))
-    )
-    (fp_circle (center 0 0) (end 2.45 0) (layer F.CrtYd) (width 0.05))
-    (fp_circle (center 0 0) (end 2.2 0) (layer Cmts.User) (width 0.15))
-    (fp_text user %R (at 0.3 0) (layer F.Fab)
-      (effects (font (size 1 1) (thickness 0.15)))
-    )
-    (pad 1 thru_hole circle (at 0 0) (size 4.4 4.4) (drill 2.2) (layers *.Cu *.Mask))
-  )
-  (module MountingHole:MountingHole_2.2mm_M2_Pad (layer F.Cu)
-    (at 105.56875 102.39375)
-    (descr "Mounting Hole 2.2mm, M2")
-    (tags "mounting hole 2.2mm m2")
-    (attr virtual)
-    (fp_text reference REF** (at 0 -3.2) (layer F.SilkS) hide
-      (effects (font (size 1 1) (thickness 0.15)))
-    )
-    (fp_text value MountingHole_2.2mm_M2_Pad (at 0 3.2) (layer F.Fab)
-      (effects (font (size 1 1) (thickness 0.15)))
-    )
-    (fp_circle (center 0 0) (end 2.45 0) (layer F.CrtYd) (width 0.05))
-    (fp_circle (center 0 0) (end 2.2 0) (layer Cmts.User) (width 0.15))
-    (fp_text user %R (at 0.3 0) (layer F.Fab)
-      (effects (font (size 1 1) (thickness 0.15)))
-    )
-    (pad 1 thru_hole circle (at 0 0) (size 4.4 4.4) (drill 2.2) (layers *.Cu *.Mask))
-  )
   (module Diode_SMD:D_SOD-123 (layer B.Cu)
     (at 334.9625 152.4 90)
@@
     (pad S2 smd rect (at 2.8 -3.875) (size 1.2 1.8) (layers B.Cu B.Paste B.Mask)
       (net 1 GND))
+    (model "D:/Keyboard Design/PCBs/TheStrkr/FTRM60/lib/JST/SM04B-SRSS-TB(LF)(SN)--3DModel-STEP-56544.STEP"
+      (offset (xyz 0 -0.5 -0.25))
+      (scale (xyz 1 1 1))
+      (rotate (xyz -90 0 0))
+    )
   )
   (module MX_Only:MXOnly-1U-NoLED (layer F.Cu)
@@
   (segment (start 158.37 165.0375) (end 158.75 165.0375) (width 0.254) (layer B.Cu) (net 20))
   (segment (start 153.3525 160.02) (end 158.37 165.0375) (width 0.254) (layer B.Cu) (net 20))
-  (segment (start 272.1475 161.4375) (end 275.01625 164.30625) (width 0.254) (layer B.Cu) (net 21))
-  (segment (start 282.97275 164.30625) (end 283.38125 163.89775) (width 0.254) (layer B.Cu) (net 21))
-  (segment (start 283.38125 163.89775) (end 283.38125 162.86875) (width 0.254) (layer B.Cu) (net 21))
-  (segment (start 275.01625 164.30625) (end 282.97275 164.30625) (width 0.254) (layer B.Cu) (net 21))
-  (segment (start 269.80375 161.90625) (end 270.2725 161.4375) (width 0.254) (layer B.Cu) (net 22))
-  (segment (start 259.7 161.90625) (end 269.80375 161.90625) (width 0.254) (layer B.Cu) (net 22))
-  (segment (start 283.51874 164.76026) (end 284.38125 163.89775) (width 0.254) (layer B.Cu) (net 23))
-  (segment (start 272.1475 163.4375) (end 273.47026 164.76026) (width 0.254) (layer B.Cu) (net 23))
-  (segment (start 284.38125 163.89775) (end 284.38125 162.86875) (width 0.254) (layer B.Cu) (net 23))
-  (segment (start 273.47026 164.76026) (end 283.51874 164.76026) (width 0.254) (layer B.Cu) (net 23))
-  (segment (start 269.786973 162.951973) (end 270.2725 163.4375) (width 0.254) (layer B.Cu) (net 24))
-  (segment (start 269.533229 162.698229) (end 269.786973 162.951973) (width 0.254) (layer B.Cu) (net 24))
-  (segment (start 263.45417 162.698229) (end 269.533229 162.698229) (width 0.254) (layer B.Cu) (net 24))
-  (segment (start 263.446149 162.70625) (end 263.45417 162.698229) (width 0.254) (layer B.Cu) (net 24))
-  (segment (start 259.7 162.70625) (end 263.446149 162.70625) (width 0.254) (layer B.Cu) (net 24))
+  (segment (start 283.65625 163.61875) (end 283.65625 163.70055) (width 0.2) (layer B.Cu) (net 21))
+  (segment (start 283.38125 163.34375) (end 283.65625 163.61875) (width 0.2) (layer B.Cu) (net 21))
+  (segment (start 283.38125 162.86875) (end 283.38125 163.34375) (width 0.2) (layer B.Cu) (net 21))
+  (segment (start 283.65625 163.70055) (end 283.27555 164.08125) (width 0.2) (layer B.Cu) (net 21))
+  (segment (start 273.829302 163.119302) (end 272.1475 161.4375) (width 0.2) (layer B.Cu) (net 21))
+  (segment (start 283.27555 164.08125) (end 274.79125 164.08125) (width 0.2) (layer B.Cu) (net 21))
+  (segment (start 274.79125 164.08125) (end 273.829302 163.119302) (width 0.2) (layer B.Cu) (net 21))
+  (segment (start 269.786973 161.923027) (end 259.716777 161.923027) (width 0.254) (layer B.Cu) (net 22))
+  (segment (start 259.716777 161.923027) (end 259.7 161.90625) (width 0.254) (layer B.Cu) (net 22))
+  (segment (start 270.2725 161.4375) (end 269.786973 161.923027) (width 0.254) (layer B.Cu) (net 22))
+  (segment (start 284.38125 163.34375) (end 284.10625 163.61875) (width 0.2) (layer B.Cu) (net 23))
+  (segment (start 284.38125 162.86875) (end 284.38125 163.34375) (width 0.2) (layer B.Cu) (net 23))
+  (segment (start 284.10625 163.61875) (end 284.10625 163.88695) (width 0.2) (layer B.Cu) (net 23))
+  (segment (start 284.10625 163.88695) (end 283.46195 164.53125) (width 0.2) (layer B.Cu) (net 23))
+  (segment (start 283.46195 164.53125) (end 274.604853 164.53125) (width 0.2) (layer B.Cu) (net 23))
+  (segment (start 274.604853 164.53125) (end 273.511103 163.4375) (width 0.2) (layer B.Cu) (net 23))
+  (segment (start 273.511103 163.4375) (end 272.1475 163.4375) (width 0.2) (layer B.Cu) (net 23))
+  (segment (start 260.704 162.70625) (end 259.7 162.70625) (width 0.254) (layer B.Cu) (net 24))
+  (segment (start 260.712021 162.698229) (end 260.704 162.70625) (width 0.254) (layer B.Cu) (net 24))
+  (segment (start 269.533229 162.698229) (end 260.712021 162.698229) (width 0.254) (layer B.Cu) (net 24))
+  (segment (start 270.2725 163.4375) (end 269.533229 162.698229) (width 0.254) (layer B.Cu) (net 24))
   (segment (start 246 159.01025) (end 246 158.925) (width 0.254) (layer B.Cu) (net 25))
   (segment (start 247.296 160.30625) (end 246 159.01025) (width 0.254) (layer B.Cu) (net 25))
@@
   (segment (start 328.6125 88.8375) (end 328.6125 88.1335) (width 0.254) (layer B.Cu) (net 70))
   (segment (start 339.09 83.82) (end 348.615 83.82) (width 0.254) (layer B.Cu) (net 70))
-  (segment (start 348.516599 106.139911) (end 351.78651 102.87) (width 0.254) (layer B.Cu) (net 71))
-  (segment (start 348.516599 107.095901) (end 348.516599 106.139911) (width 0.254) (layer B.Cu) (net 71))
-  (segment (start 346.460499 109.152001) (end 348.516599 107.095901) (width 0.254) (layer B.Cu) (net 71))
   (segment (start 351.78651 102.87) (end 353.3775 102.87) (width 0.254) (layer B.Cu) (net 71))
-  (segment (start 339.491751 109.152001) (end 346.460499 109.152001) (width 0.254) (layer B.Cu) (net 71))
-  (segment (start 338.93125 108.5915) (end 339.491751 109.152001) (width 0.254) (layer B.Cu) (net 71))
-  (segment (start 338.93125 107.8875) (end 338.93125 108.5915) (width 0.254) (layer B.Cu) (net 71))
+  (segment (start 343.24475 102.87) (end 351.78651 102.87) (width 0.254) (layer B.Cu) (net 71))
+  (segment (start 338.93125 107.1835) (end 343.24475 102.87) (width 0.254) (layer B.Cu) (net 71))
+  (segment (start 338.93125 107.8875) (end 338.93125 107.1835) (width 0.254) (layer B.Cu) (net 71))
   (segment (start 334.5825 150.75) (end 334.9625 150.75) (width 0.254) (layer B.Cu) (net 72))
   (segment (start 329.565 145.7325) (end 334.5825 150.75) (width 0.254) (layer B.Cu) (net 72))
@@
     (connect_pads (clearance 0.508))
     (min_thickness 0.254)
-    (fill yes (arc_segments 32) (thermal_gap 0.508) (thermal_bridge_width 0.508))
+    (fill (arc_segments 32) (thermal_gap 0.508) (thermal_bridge_width 0.508))
     (polygon
       (pts
@@
     (connect_pads (clearance 0.508))
     (min_thickness 0.254)
-    (fill yes (arc_segments 32) (thermal_gap 0.508) (thermal_bridge_width 0.508))
+    (fill (arc_segments 32) (thermal_gap 0.508) (thermal_bridge_width 0.508))
     (polygon
       (pts
